File: Hardware/keyboard_v2/keyboard_v2.kicad_pcb (KiCad board)
At the start: 2 copper layers, 21 parts, among them J1 Conn_01x08_Male, SW1 SW_Push, SW2 SW_Push, SW3 SW_Push, SW4 SW_Push, SW5 SW_Push, SW6 SW_Push, U1 74HC14

Commit message: Распаян модуль keyboard_v2/
Parts:
- added C1: CP, Capacitor_THT:CP_Radial_D5.0mm_P2.50mm, F.Cu at (139.6, 61.3)
- added C1: CP, Capacitor_THT:CP_Radial_D5.0mm_P2.50mm, F.Cu at (88.1, 61.7)
- added C2: C, Capacitor_SMD:C_1206_3216Metric_Pad1.33x1.80mm_HandSolder, F.Cu at (147.9, 65.8)
- added C2: C, Capacitor_SMD:C_1206_3216Metric_Pad1.33x1.80mm_HandSolder, F.Cu at (96.5, 66.2)
- added C3: C, Capacitor_SMD:C_1206_3216Metric_Pad1.33x1.80mm_HandSolder, F.Cu at (158.0, 65.8)
- added C3: C, Capacitor_SMD:C_1206_3216Metric_Pad1.33x1.80mm_HandSolder, F.Cu at (106.6, 66.2)
- added C4: C, Capacitor_SMD:C_1206_3216Metric_Pad1.33x1.80mm_HandSolder, F.Cu at (168.0, 65.8)
- added C4: C, Capacitor_SMD:C_1206_3216Metric_Pad1.33x1.80mm_HandSolder, F.Cu at (116.6, 66.2)
- added C5: C, Capacitor_SMD:C_1206_3216Metric_Pad1.33x1.80mm_HandSolder, F.Cu at (167.8, 39.7)
- added C5: C, Capacitor_SMD:C_1206_3216Metric_Pad1.33x1.80mm_HandSolder, F.Cu at (116.4, 40.1)
- added C6: C, Capacitor_SMD:C_1206_3216Metric_Pad1.33x1.80mm_HandSolder, F.Cu at (158.1, 39.7)
- added C6: C, Capacitor_SMD:C_1206_3216Metric_Pad1.33x1.80mm_HandSolder, F.Cu at (106.7, 40.1)
- added C7: C, Capacitor_SMD:C_1206_3216Metric_Pad1.33x1.80mm_HandSolder, F.Cu at (147.5, 39.7)
- added C7: C, Capacitor_SMD:C_1206_3216Metric_Pad1.33x1.80mm_HandSolder, F.Cu at (96.0, 40.1)
- added J1: Conn_01x08_Male, Connector_PinHeader_2.54mm:PinHeader_1x08_P2.54mm_Vertical, F.Cu at (137.3, 38.4)
- added J1: Conn_01x08_Male, Connector_PinHeader_2.54mm:PinHeader_1x08_P2.54mm_Vertical, F.Cu at (85.9, 38.8)
- added R1: R, Resistor_SMD:R_1206_3216Metric_Pad1.30x1.75mm_HandSolder, F.Cu at (143.9, 62.3)
- added R1: R, Resistor_SMD:R_1206_3216Metric_Pad1.30x1.75mm_HandSolder, F.Cu at (92.5, 62.7)
- added R2: R, Resistor_SMD:R_1206_3216Metric_Pad1.30x1.75mm_HandSolder, F.Cu at (153.9, 62.3)
- added R2: R, Resistor_SMD:R_1206_3216Metric_Pad1.30x1.75mm_HandSolder, F.Cu at (102.5, 62.7)
- added R3: R, Resistor_SMD:R_1206_3216Metric_Pad1.30x1.75mm_HandSolder, F.Cu at (164.0, 62.3)
- added R3: R, Resistor_SMD:R_1206_3216Metric_Pad1.30x1.75mm_HandSolder, F.Cu at (112.5, 62.7)
- added R4: R, Resistor_SMD:R_1206_3216Metric_Pad1.30x1.75mm_HandSolder, F.Cu at (162.9, 35.9)
- added R4: R, Resistor_SMD:R_1206_3216Metric_Pad1.30x1.75mm_HandSolder, F.Cu at (111.5, 36.2)
- added R5: R, Resistor_SMD:R_1206_3216Metric_Pad1.30x1.75mm_HandSolder, F.Cu at (153.0, 35.9)
- added R5: R, Resistor_SMD:R_1206_3216Metric_Pad1.30x1.75mm_HandSolder, F.Cu at (101.6, 36.2)
- added R6: R, Resistor_SMD:R_1206_3216Metric_Pad1.30x1.75mm_HandSolder, F.Cu at (142.9, 35.9)
- added R6: R, Resistor_SMD:R_1206_3216Metric_Pad1.30x1.75mm_HandSolder, F.Cu at (91.4, 36.2)
- added SW1: SW_Push, Button_Switch_SMD:SW_SPST_SMD_6.4_3.7_v2, F.Cu at (148.0, 60.7)
- added SW1: SW_Push, Button_Switch_SMD:SW_SPST_SMD_6.4_3.7_v2, F.Cu at (96.5, 61.0)
- added SW2: SW_Push, Button_Switch_SMD:SW_SPST_SMD_6.4_3.7_v2, F.Cu at (158.0, 60.7)
- added SW2: SW_Push, Button_Switch_SMD:SW_SPST_SMD_6.4_3.7_v2, F.Cu at (106.5, 61.0)
- added SW3: SW_Push, Button_Switch_SMD:SW_SPST_SMD_6.4_3.7_v2, F.Cu at (167.9, 60.7)
- added SW3: SW_Push, Button_Switch_SMD:SW_SPST_SMD_6.4_3.7_v2, F.Cu at (116.5, 61.0)
- added SW4: SW_Push, Button_Switch_SMD:SW_SPST_SMD_6.4_3.7_v2, F.Cu at (167.8, 34.4)
- added SW4: SW_Push, Button_Switch_SMD:SW_SPST_SMD_6.4_3.7_v2, F.Cu at (116.3, 34.7)
- added SW5: SW_Push, Button_Switch_SMD:SW_SPST_SMD_6.4_3.7_v2, F.Cu at (158.0, 34.4)
- added SW5: SW_Push, Button_Switch_SMD:SW_SPST_SMD_6.4_3.7_v2, F.Cu at (106.5, 34.7)
- added SW6: SW_Push, Button_Switch_SMD:SW_SPST_SMD_6.4_3.7_v2, F.Cu at (147.6, 34.4)
- added SW6: SW_Push, Button_Switch_SMD:SW_SPST_SMD_6.4_3.7_v2, F.Cu at (96.2, 34.7)
- added U1: 74HC14, Package_SO:SOIC-14_3.9x8.7mm_P1.27mm, F.Cu at (157.4, 48.8)
- added U1: 74HC14, Package_SO:SOIC-14_3.9x8.7mm_P1.27mm, F.Cu at (105.9, 49.2)
- C2, C3, C4, C5, C6, C7: footprint Capacitor_SMD:C_0805_2012Metric_Pad1.18x1.45mm_HandSolder -> Capacitor_SMD:C_1206_3216Metric_Pad1.33x1.80mm_HandSolder
- SW1, SW2, SW3, SW4, SW5, SW6: footprint Button_Switch_SMD:SW_SPST_SMD_6.4_3.7 -> Button_Switch_SMD:SW_SPST_SMD_6.4_3.7_v2
- moved C1 62.1 mm to (37.3, 61.7)
- moved C3 62.1 mm to (55.8, 66.3)
- moved C5 62.1 mm to (65.6, 40.1)
- moved C6 62.1 mm to (55.9, 40.1)
- moved C7 62.1 mm to (45.2, 40.1)
- moved J1 62.1 mm to (35.1, 38.9)
- moved R4 62.1 mm to (60.7, 36.3)
- moved R5 62.1 mm to (50.8, 36.3)
- moved R6 62.1 mm to (40.6, 36.3)
- moved SW1 62.1 mm to (45.7, 61.1)
- moved SW2 62.1 mm to (55.7, 61.1)
- moved SW3 62.1 mm to (65.7, 61.1)
- moved SW4 62.1 mm to (65.5, 34.8)
- moved SW5 62.1 mm to (55.7, 34.8)
- moved C2 62.1 mm to (45.7, 66.3)
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Routing:
- net (no net): track 153.7 -> 701.5 mm
- net GND: track 207.1 -> 15.9 mm
- net Net-(C4-Pad1): track 15.1 -> 13.8 mm
- net Net-(C3-Pad1): track 10.7 -> 9.48 mm
- net Net-(C5-Pad1): track 15.7 -> 14.6 mm
- net Net-(C2-Pad1): track 14.5 -> 13.4 mm
- added copper zone on F.Cu, net (none)
- added copper zone on F.Cu, net GND
