File: Hardware/All-in-one/All-in-one.sch (KiCad schematic (older format))
At the start: 10 parts, among them J1 Conn_01x04_Male, J2 Barrel_Jack, J3 Micro_SD_Card, SW1 SW_Push, U1 DHT11, U2 BME280_module, U3 YAAJ_BluePill_Part_Like_SWD_B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

Commit message: Схема электрическая принципиальная All-in-one/
Parts:
- removed J3: Micro_SD_Card, symbol Connector:Micro_SD_Card
- removed SW1: SW_Push, symbol Switch:SW_Push
- removed U2: BME280_module, symbol megasaturnv_custom_components:BME280_module
- added J4, J5, J6, J7, J8: Conn_01x02_Male, Connector_PinHeader_2.54mm:PinHeader_1x02_P2.54mm_Vertical, symbol Connector:Conn_01x02_Male
- added U2: BMP280_flipped, megasaturnv_custom_components:BMP280_flipped, symbol megasaturnv_custom_components:BMP280_flipped
- added U4: microSD_flipped, megasaturnv_custom_components:microSD_Card_3V3, symbol megasaturnv_custom_components:microSD_flipped
- J1: footprint (none) -> Connector_PinHeader_2.54mm:PinHeader_1x04_P2.54mm_Vertical
- J2: footprint (none) -> Connector_BarrelJack:BarrelJack_Horizontal
- R1, R2: footprint (none) -> Resistor_THT:R_Axial_DIN0207_L6.3mm_D2.5mm_P7.62mm_Horizontal
- RTC1: footprint (none) -> megasaturnv_custom_components:RTC_DS3231; symbol megasaturnv_custom_components:RTC_DS3231 -> All-in-one-rescue:RTC_DS3231-megasaturnv_custom_components
- U3: footprint (none) -> Footprints:YAAJ_BluePill_SWD_1; symbol YAAJ_BluePill_Part_Like_SWD_Breakout:YAAJ_BluePill_Part_Like_SWD_Breakout -> All-in-one-rescue:YAAJ_BluePill_Part_Like_SWD_Breakout-YAAJ_BluePill_Part_Like_SWD_Breakout
Connections:
- net I2C1_SCL: now reaches U3.14 (PB6)
- net I2C1_SCL: now also J1.2 (Pin_2), RTC1.4 (SCL), U2.4 (SCL)
- net I2C1_SDA: now reaches U3.15 (PB7)
- net I2C1_SDA: now also J1.1 (Pin_1), RTC1.3 (SDA), U2.3 (SDA)
- net +5V: now reaches U3.18 (5V)
- net +5V: now also J1.3 (Pin_3), J2.1, RTC1.2 (VCC), J4.2 (Pin_2), J5.2 (Pin_2)
- net GND: now reaches U3.19 (GND)
- net GND: now also J1.4 (Pin_4), J2.2, RTC1.1 (GND), J4.1 (Pin_1), J5.1 (Pin_1), J7.2 (Pin_2), J8.1 (Pin_1), U2.1 (SDO), U2.5 (GND), U4.1 (GND)
- net 3V3: now reaches U3.20 (3V3)
- net 3V3: now also R1.1, R2.1, U2.2 (CBS), U2.6 (VCC), U4.6 (3V3)
- net A1: now reaches U3.26 (PA1)
- net A1: now also R1.2, J7.1 (Pin_1)
- net A2: now reaches U3.27 (PA2)
- net A2: now also R2.2, J8.2 (Pin_2)
- net at U3.29 (PA4): now also U4.5 (CS)
- net at U3.30 (PA5): now also U4.3 (CLK)
- net at U3.31 (PA6): now also U4.2 (MISO)
- net at U3.32 (PA7): now also U4.4 (MOSI)
- net at U3.35 (PB10): now also J6.1 (Pin_1)
- net at U3.36 (PB11): now also J6.2 (Pin_2)
Other:
- moved on the sheet: J1, J2, R1, R2, RTC1, U1
