File: Hardware/All-in-one/_autosave-All-in-one.sch (KiCad schematic (older format))
At the start: 14 parts, among them J1 Conn_01x04_Male, J2 Barrel_Jack, J3 Conn_01x03, J4 Conn_01x02_Male, J5 Conn_01x02_Male, J7 Conn_01x02_Male, J8 Conn_01x02_Male, U2 BMP280_flipped, U3 YAAJ_BluePill_Part_Like, U4 microSD_flipped

Commit message: Продолжаем разводить п.п. На морозе часы неожиданно сбросились. справлени баг со слишком ранним выходом из режима настройки часов. 30 секунд недостаточно, чтобы точно сбросить секунды
Parts:
- gave numbers to parts that had none: 1
Changed lines of the file:
@@
 3V3
 $Comp
-L Connector_Generic:Conn_01x03 J?
+L Connector_Generic:Conn_01x03 J6
 U 1 1 602FFCC0
 P 2850 2500
-F 0 "J?" H 2930 2542 50  0000 L CNN
+F 0 "J6" H 2930 2542 50  0000 L CNN
 F 1 "Conn_01x03" H 2930 2451 50  0000 L CNN
 F 2 "Connector_PinHeader_2.54mm:PinHeader_1x03_P2.54mm_Vertical" H 2850 2500 50  0001 C CNN
@@
 3V3
 $Comp
-L power:GND #PWR?
+L power:GND #PWR0105
 U 1 1 6030D641
 P 3200 2700
-F 0 "#PWR?" H 3200 2450 50  0001 C CNN
+F 0 "#PWR0105" H 3200 2450 50  0001 C CNN
 F 1 "GND" H 3205 2527 50  0000 C CNN
 F 2 "" H 3200 2700 50  0001 C CNN
